Commit message: add depth-range usage for stereo Tracking

File: toBeAdded_freeFloatDemo/urdf/arm5e_B.xacro (robot description, xacro)
@@ -2,5 +2,4 @@
 <robot name="arm5e_A" xmlns:xacro="http://www.ros.org/wiki/xacro">
   <xacro:property name="pi" value="3.1415926535897931"/>
-  <xacro:property name="pi" value="3.141592654" />
   <xacro:property name="robot_parts_path" value="robot/ARM5E/ARM5E" />
   <xacro:property name="ext" value="osg" />
@@ -125,9 +124,11 @@
     <buoyancy><compensation>1.0</compensation></buoyancy>
   </link>
-    <joint name="JawRotate" type="continuous">
+    <joint name="JawRotate" type="revolute">
     <parent link="part3"/>
     <child link="part4_base"/>
     <axis xyz="0 0 1"/>
     <origin rpy="${pi/2} 0 ${theta2}" xyz="${0.083/cos180minusTheta2+sin180minusTheta2*0.1485} ${cos180minusTheta2*0.1485} 0"/>
+    <dynamics damping="0.8"/>
+    <limit lower="${-pi}" upper="${pi}" velocity="1" effort="200"/>
     </joint>
       <link name="end_effector"> <!-- From the kinematic base of the robot -->

File: toBeAdded_freeFloatDemo/urdf/g500ARM5BPeg_uwsim.urdf (robot description, URDF)
Before this commit: robot g500_B, 10 links, 9 joints
Joints:
- joint JawRotate: limit (none) -> lower=-3.14159265359 upper=3.14159265359 effort=200 velocity=1; origin xyz=0.349117258152 0.058023572508 0 rpy=1.570796327 0 1.972222055 -> xyz=0.349117258152 0.058023572508 0 rpy=1.57079632679 0 1.972222055; type continuous -> revolute
- joint Shoulder: origin xyz=0.08052 0 0 rpy=1.570796327 0 0 -> xyz=0.08052 0 0 rpy=1.57079632679 0 0
- joint Slew: limit lower=-1.570796327 upper=0.5488 effort=500 velocity=1 -> lower=-1.57079632679 upper=0.5488 effort=500 velocity=1
- joint baselink_to_part0: origin xyz=0 0 0.95 rpy=0 0 3.141592654 -> xyz=0 0 0.95 rpy=0 0 3.14159265359
